File: KiKad_Project/PCB_Card.kicad_pcb (KiCad board)
At the start: 2 copper layers, 88 x 55 mm, 70 parts, among them J1 USB_B_Micro, J10 SD_Card, J2 EXT_SPI, J3 GPIO, J4 EXT_I2C, J5 EXT_UART, J6 Conn_01x12_Female, J9 SWD, Q1 NTR4003, SW1 Power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

Commit message: Updated to latest PCB CAD (revision 3)
Parts:
- removed the G*** at (135.7, 81.5) (x2)
- added G***: LOGO, PCB_Graphics:Oxford_Logo_35mm_Mask, F.Cu at (135.8, 81.8)
- added G***: LOGO, PCB_Graphics:Oxford_Logo_35mm_Silk, F.Cu at (135.8, 81.8)
- added G***: LOGO, PCB_Graphics:Oxford_Logo_35mm_Copper, F.Cu at (135.8, 81.8)
- added R11: 33K, Resistor_SMD:R_0805_2012Metric_Pad1.15x1.40mm_HandSolder, F.Cu at (187.1, 100.3)
- added TP10: D-, Alex_Parts:TestPoint_Pad_D1.0mm, B.Cu at (186.4, 78.0)
- added TP7: TestPoint, TestPoint:TestPoint_THTPad_D2.0mm_Drill1.0mm, F.Cu at (162.0, 91.0)
- added TP8: +5V, TestPoint:TestPoint_Pad_D3.0mm, B.Cu at (167.4, 76.7)
- added TP9: D+, Alex_Parts:TestPoint_Pad_D1.0mm, B.Cu at (184.4, 80.5)
- Q1: value NTR4003 -> BC817DS; footprint Package_TO_SOT_SMD:SOT-23 -> Package_TO_SOT_SMD:SOT-23-6_Handsoldering
- R14: value 82R -> 6R8
- R4: value 82R -> 22R
- R5: value 82R -> 120R
- R6: value 82R -> 16R
- R9: value 33K -> 1K5
- Y1: footprint Crystal:Crystal_SMD_5032-4Pin_5.0x3.2mm -> Crystal:Crystal_SMD_Abracon_ABM3-2Pin_5.0x3.2mm_HandSoldering
- moved TP6 10.4 mm to (161.6, 108.9)
- moved R14 9.62 mm to (174.9, 107.1), turned to 180 degrees
- moved TP4 6.40 mm to (163.3, 106.3)
- moved TP3 4.39 mm to (164.4, 105.4)
- moved C6 3.05 mm to (164.9, 101.8), turned to 270 degrees
- moved TP2 2.42 mm to (165.5, 104.5)
- moved TP5 2.15 mm to (164.6, 97.0)
- moved R9 1.86 mm to (174.9, 103.9), turned to 0 degrees
- moved Q1 1.66 mm to (170.1, 106.0)
- moved C8 1.65 mm to (186.1, 107.1), turned to 0 degrees
- moved C7 1.57 mm to (178.6, 107.1), turned to 180 degrees
- moved TP1 1.41 mm to (163.7, 98.2)
- moved Y1 1.39 mm to (182.3, 104.2)
- moved JP1 0.97 mm to (162.0, 88.3)
- moved JP2 0.63 mm to (162.0, 93.7)
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Connections:
- D2 pad 1: +5V -> +3V3
- Q1 pad 1: LCD_LED_CTRL -> Net-(Q1-Pad1)
- Q1 pad 2: GND -> Net-(Q1-Pad2)
- Q1 pad 3: Net-(Q1-Pad3) -> Net-(Q1-Pad2)
- R14 pad 1: Net-(J6-Pad2) -> GND
- R14 pad 2: Net-(Q1-Pad3) -> Net-(Q1-Pad1)
- R9 pad 1: LCD_LED_CTRL -> Net-(Q1-Pad2)
- R9 pad 2: GND -> LCD_LED_CTRL
- U1 pad 40: LCD_DC -> LCD_RST
- U1 pad 41: LCD_RST -> LCD_DC
- Y1 pad 2: Net-(Y1-Pad2) -> OSC_2
Routing:
- net +3V3: track 227.3 -> 261.4 mm, vias 12 -> 13
- net BOOT0: track 22.7 -> 56.2 mm, vias 2 -> 4
- net +5V: track 230.2 -> 209.7 mm, vias 4 -> 5
- net LCD_RST: track 10.5 -> 22.7 mm
- net Net-(J6-Pad2): track 3.65 -> 15.0 mm, vias 0 -> 2
- net GND: track 398.9 -> 392.6 mm, vias 9 -> 10
- net OSC_1: track 16.0 -> 10.2 mm
- net Net-(Q1-Pad1): track 0.00 -> 5.82 mm
- net Net-(Q1-Pad2): track 0.00 -> 5.42 mm
- net Net-(Q1-Pad3): track 4.84 -> 0.00 mm
- net EXT_UART_RX: track 34.4 -> 37.1 mm, vias 2 -> 0
- net LCD_LED_CTRL: track 35.0 -> 37.5 mm
- net LCD_CS: track 22.8 -> 25.3 mm
- net LED_G: track 40.1 -> 37.9 mm
- net GPIO_PA9: track 24.8 -> 26.9 mm
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Other:
- board text added: "51-G-1384-480-03"
- board text added: "PC13"
- board text added: "PC14"
- board text added: "PC15"
- board text added: "STM32F103C8T6 Breakout Board"
- board text removed: "51-G-1384-480-02"
- board text removed: "STM32F103CT8 Breakout Board"
