File: KiKad_Project/PCB_Card.sch (KiCad schematic (older format))
At the start: 57 parts, among them J1 USB_B_Micro, J10 SD_Card, J2 EXT_SPI, J3 GPIO, J4 EXT_I2C, J5 EXT_UART, J6 Conn_01x12_Female, J9 SWD, Q1 NTR4003, SW1 Power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

Commit message: Updated to latest PCB CAD (revision 3)
Parts:
- removed Q1: NTR4003, Package_TO_SOT_SMD:SOT-23, symbol Device:Q_NMOS_GSD
- removed Y1: 8MHz, Crystal:Crystal_SMD_5032-4Pin_5.0x3.2mm, symbol Device:Crystal_GND2
- added Q1: BC817DS, Package_TO_SOT_SMD:SOT-23-6_Handsoldering, symbol Device:Q_DUAL_NPN_NPN_E1B1C2E2B2C1
- added R11: 33K, Resistor_SMD:R_0805_2012Metric_Pad1.15x1.40mm_HandSolder, symbol Device:R
- added TP10: D-, Alex_Parts:TestPoint_Pad_D1.0mm, symbol Connector:TestPoint
- added TP7: TestPoint, TestPoint:TestPoint_THTPad_D2.0mm_Drill1.0mm, symbol Connector:TestPoint
- added TP8: +5V, TestPoint:TestPoint_Pad_D3.0mm, symbol Connector:TestPoint
- added TP9: D+, Alex_Parts:TestPoint_Pad_D1.0mm, symbol Connector:TestPoint
- added Y1: 8MHz, Crystal:Crystal_SMD_Abracon_ABM3-2Pin_5.0x3.2mm_HandSoldering, symbol Device:Crystal
- J10: symbol Connector:Micro_SD_Card_Det_Hirose_DM3AT -> PCB_Card-rescue:Micro_SD_Card_Det_Hirose_DM3AT-Connector
- R14: value 82R -> 6R8
- R4: value 82R -> 22R
- R5: value 82R -> 120R
- R6: value 82R -> 16R
- R9: value 33K -> 1K5
Connections:
- net +3V3: now also D2.1 (A)
- net +5V: now also TP8.1; no longer D2.1 (A)
- net BOOT0: now also R11.1, TP7.1
- net GND: now also R14.1, Q1.4 (E2), R11.2; no longer R9.2
- net LCD_DC: now also U1.41 (PB5); no longer U1.40 (PB4)
- net LCD_LED_CTRL: now also R9.2; no longer R9.1
- net LCD_RST: now also U1.40 (PB4); no longer U1.41 (PB5)
- net OSC_1: now also Y1.1
- net OSC_2: now also Y1.2
- net USB_D+: now also TP9.1
- net USB_D-: now also TP10.1
- net at J6.2 (Pin_2): now also Q1.6 (C1); no longer R14.1
- net at R14.2: now also Q1.1 (E1), Q1.5 (B2)
- new net: Q1.2 (B1), Q1.3 (C2), R9.1
- no-connect marks 6 -> 5
Other:
- moved on the sheet: BT1, C1, C10, C11, C2, C3, C4, C5, C6, C7, C8, C9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
